File: PCB/Buck Converter Tester.kicad_pcb (KiCad board)
At the start: 2 copper layers, 99.5 x 65 mm, 11 parts, among them J1 Conn_01x07_Male, J2 Conn_01x11_Male, J3 Conn_01x07_Male

Commit message: images
Routing:
- removed copper zone on B.Cu, net +5V
- removed copper zone on B.Cu, net VCC
